File: IO.kicad_sch (KiCad schematic)
At the start: 5 parts, among them J1 Conn_02x10_Odd_Even, J2 Conn_01x08, J3 Conn_01x08

Commit message: Small edit
Parts:
- H1, H2: value MountingHole -> (none)
- J1: value Conn_02x10_Odd_Even -> (none)
- J2, J3: value Conn_01x08 -> (none)
Other:
- note removed: "INTERFACING WITH OTHER HIERARCHIES ONLY WITH HIERARCHICAL LABEL"
- moved on the sheet: H1, H2, J1
